File: embeddeds/gwaamc training aid.sch (KiCad schematic (older format))
At the start: 18 parts, among them J1 Conn_Coaxial, U1 LM334Z, U1-LSB MCP4162-502(0-5KΩ), U1-MSBs... MCP4162-104(0-100KΩ), U2 LM334Z, U2-LSB MCP4162-502(0-5KΩ), U2-MSBs... MCP4162-104(0-100KΩ), U3-A AD8244ARMZ, U3-B AD8244ARMZ, U3-C AD8244ARMZ, U3-D AD8244ARMZ, U4 74LV138

Commit message: Schematic created in KiCad
Parts:
- added U4: 74LV138 only needed with larger numbers of DPots, symbol 74xx:74LS138
- ADC1: value HX711 or ADS1X15 -> HX711, etc.
- C1_bank: renamed from C1; value 0.05 µF -> 2.05 µF total
- C2_bank: renamed from C2; value 0.05 µF -> 2.05 µF total
- U3-A: value AD8244ARMZ -> (none)
- U3-B, U3-C, U3-D: value AD8244ARMZ -> U3_AD8244ARMZ
- U5...: renamed from U4; value 74LV138 -> 74LV138 only for large numbers of DPots
- renumbered U1-LSB to DPot1-LSB, U1-MSBs... to DPot1-MSBs..., U2-LSB to DPot2-LSB, U2-MSBs... to DPot2-MSBs..., Electrodes_contacting_plant_leaf to Electrodes_contacting_plant_leaf_surfaces
Connections:
- net labels added: -LEAF-, <Drives_DPot_CS_pins_when_required, <From_MCU_Digital_pins_alternate_method_to_DPot_CS_pins, Earth_Protective, Opt_SW, Unused_leaf, coaxial_cable
- net labels removed: Coaxial_cable
- wire segments 68 -> 90
Other:
- note added: "(Switch wiring overlaps straight-through \nwiring for drawing purposes only. Do not \nwire both ways simultaneously, of course)"
- note added: "*See note"
- note added: "*See note for the above DPot set"
- note added: "18 Dec 2018"
- note added: "DUT stem"
- note added: "Device Under Test \n(DUT)"
- note added: "NOTE FOR MCU ANALOG PINS: User-\npreference allowed in preprocessor \nmacros for additional traces from \nunused Analog Pins."
- note added: "NOTE: Arduino also gets power rails \nand a serial connection to a computer"
- note added: "NOTE: Decoupling C banks 1-2 each consist of a \n2-10 µF tantalum plus a low-ESR sub-µF capacitor \nwhich gets located in direct-as-practical path \nbetween + and GND pins of the active device \npaired with."
- note added: "NOTE: If convenient polarity flipping is desired,\n a 4-way house light switch may be placed in \nthe electrode circuit between the electrodes and the \ncoaxial cable, assuming you hook it up correctly."
- note added: "NOTE: The LM334 devices must receive 5 VDC or greater due to their own operating voltage range. \nTheir functional range will be substantially limited if powered by the 3 or 3.3 VDC of many MCUs. \nProvide a dedicated positive power supply to them if 5 VDC is not otherwise available, and carefully \nensure the output levels from them are prevented from exceeding the input range of the remaining \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"
- note added: "NOTE: U5 only used for larger numbers of DPots. U5's outputs drive DPot CS lines. U4 only used for even \nlarger numbers of DPots. U4's outputs drive E1 or E2 of U5, U6, U7, etc. See sketch preprocessor macros \nand comments for more complete pin assignments and requirements.\nU5 pin E1/E2 may be driven by an MCU Digital Pin. Again, see sketch comments."
- note added: "NOTE: Unfortunately, the devices shown do \nnot all share common data protocols except \nthe DPots. Define the Digital Pin functions \nin preprocessor macros for all the disparate\nprotocols. Some flexibility thus remains for \ndriving an additional device or two that may \nhave inflexible pin assignments."
- note added: "Twisted pair with \noptional 4-way switch \ninserted to flip polarity"
- note removed: "17 Dec 2018"
- note removed: "Arduino gets power and a \nserial connection to a computer"
- note removed: "NOTE: Devices shown all do not share \ndata over the same Digital Pins except\nthat all DPots share their SCK lines and\ntheir SDI lines. Define the Digital Pin \nfunctions in preprocessor macros."
- note removed: "NOTE: If convenient polarity flipping\nis desired, a 4-way house light switch \nmay be placed in the electrode circuit\nbetween the electrodes and the coaxial\ncable, assuming you hook it up correctly."
- note removed: "NOTE: MCU=Arduino"
- note removed: "NOTE: U4 only used for large numbers \nof DPots. Its outputs drive DPot CS lines.\nSee sketch comments."
- moved on the sheet: ADC1, C1_bank, C2_bank, DPot1-LSB, DPot1-MSBs..., DPot2-LSB, DPot2-MSBs..., Electrodes_contacting_plant_leaf_surfaces, J1, MCU, R1, U1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

Commit message: Add files via upload
Connections:
- wire segments 90 -> 92
Other:
- note added: "1"
- note added: "NOTE: Unfortunately, the devices shown do \nnot all share common data protocols except \nthe DPots. Define the Digital Pin functions \nin preprocessor macros for all the disparate\nprotocols. Thus, some flexibility remains for \ndriving an additional device or two that may \nhave inflexible pin assignments."
- note added: "This system is shown using: Shown but not in use:\n1 - LM334 bridge 1 - Uno Arduino 2 - 74LV138; useful with high DPot count\n1 - HX711 24-bit ADC\n1 - LSB DPot/leg Non-LM334 configuration options include bridged and\n1 - MSB DPot/leg single leg to replace or augment LM334 option."
- note removed: "A Reviving Civility"
- note removed: "NOTE: Unfortunately, the devices shown do \nnot all share common data protocols except \nthe DPots. Define the Digital Pin functions \nin preprocessor macros for all the disparate\nprotocols. Some flexibility thus remains for \ndriving an additional device or two that may \nhave inflexible pin assignments."
- moved on the sheet: ADC1, C1_bank, C2_bank, MCU, U3-A, U3-B, U3-C, U3-D

Commit message: Add files via upload
Other:
- note added: "NOTE FOR MCU ANALOG PINS: Low-\nnumbered Analog Input pins are reserved \nfor all existing DPOT-controlled leg outputs. \nUnused Analog Pins above them may be\nused to display additional plotter traces\nwhen so defined in preprocessor macros."
- note added: "This system is shown using: Shown not being used:\n1 - LM334 bridge 1 - Uno Arduino 2 - 74LV138; useful with high DPot count\n1 - HX711 24-bit ADC\n1 - LSB DPot/leg Non-LM334 configuration options include bridged and\n1 - MSB DPot/leg single leg to replace or augment LM334 option."
- note removed: "NOTE FOR MCU ANALOG PINS: User-\npreference allowed in preprocessor \nmacros for additional traces from \nunused Analog Pins."
- note removed: "This system is shown using: Shown but not in use:\n1 - LM334 bridge 1 - Uno Arduino 2 - 74LV138; useful with high DPot count\n1 - HX711 24-bit ADC\n1 - LSB DPot/leg Non-LM334 configuration options include bridged and\n1 - MSB DPot/leg single leg to replace or augment LM334 option."
Changed lines of the file:
@@
 18 Dec 2018
 Text Notes 7000 7050 0    63   ~ 0
-This system is shown using:                Shown but not in use:\n1 - LM334 bridge   1 - Uno Arduino      2 - 74LV138; useful with high DPot count\n1 - HX711 24-bit ADC\n1 - LSB DPot/leg            Non-LM334 configuration options include bridged and\n1 - MSB DPot/leg           single leg to replace or augment LM334 option.
+This system is shown using:                Shown not being used:\n1 - LM334 bridge   1 - Uno Arduino      2 - 74LV138; useful with high DPot count\n1 - HX711 24-bit ADC\n1 - LSB DPot/leg            Non-LM334 configuration options include bridged and\n1 - MSB DPot/leg           single leg to replace or augment LM334 option.
 $Comp
 L 74xx:74LS138 U4
@@
 Text Notes 10750 5000 1    60   Italic 12
 *See note
-Text Notes 9200 6400 0    56   ~ 11
-NOTE FOR MCU ANALOG PINS:  User-\npreference allowed in preprocessor \nmacros for additional traces from \nunused Analog Pins.
+Text Notes 9150 6450 0    56   ~ 11
+NOTE FOR MCU ANALOG PINS:  Low-\nnumbered Analog Input pins are reserved \nfor all existing DPOT-controlled leg outputs.  \nUnused Analog Pins above them may be\nused to display additional plotter traces\nwhen so defined in preprocessor macros.
 Text Notes 3650 3850 0    56   ~ 0
 NOTE: Decoupling C banks 1-2 each consist of a \n2-10 µF tantalum plus a low-ESR sub-µF capacitor \nwhich gets located in direct-as-practical path \nbetween + and GND pins of the active device \npaired with.

Commit message: Add files via upload
Other:
- note added: "*NOTE FOR MCU ANALOG PINS: Low-\nnumbered Analog Input pins are reserved \nfor all existing DPOT-controlled leg outputs. \nUnused Analog Pins above them may be\nused to display additional plotter traces\nwhen so defined in preprocessor macros."
- note added: "*NOTE: U5 only used for larger numbers of DPots. U5's outputs drive DPot CS lines. U4 only used for even \nlarger numbers of DPots. U4's outputs drive E1 or E2 of U5, U6, U7, etc. See sketch preprocessor macros \nand comments for more complete pin assignments and requirements.\nU5 pin E1/E2 may be driven by an MCU Digital Pin. Again, see sketch comments."
- note removed: "NOTE FOR MCU ANALOG PINS: Low-\nnumbered Analog Input pins are reserved \nfor all existing DPOT-controlled leg outputs. \nUnused Analog Pins above them may be\nused to display additional plotter traces\nwhen so defined in preprocessor macros."
- note removed: "NOTE: U5 only used for larger numbers of DPots. U5's outputs drive DPot CS lines. U4 only used for even \nlarger numbers of DPots. U4's outputs drive E1 or E2 of U5, U6, U7, etc. See sketch preprocessor macros \nand comments for more complete pin assignments and requirements.\nU5 pin E1/E2 may be driven by an MCU Digital Pin. Again, see sketch comments."
Changed lines of the file:
@@
 $EndComp
 Text Notes 6250 1100 0    58   ~ 0
-NOTE: U5 only used for larger numbers of DPots.  U5's outputs drive DPot CS lines.  U4 only used for even \nlarger numbers of DPots.  U4's outputs drive E1 or E2 of U5, U6, U7, etc. See sketch preprocessor macros \nand comments for more complete pin assignments and requirements.\nU5 pin E1/E2 may be driven by an MCU Digital Pin.  Again, see sketch comments.
+*NOTE: U5 only used for larger numbers of DPots.  U5's outputs drive DPot CS lines.  U4 only used for even \nlarger numbers of DPots.  U4's outputs drive E1 or E2 of U5, U6, U7, etc. See sketch preprocessor macros \nand comments for more complete pin assignments and requirements.\nU5 pin E1/E2 may be driven by an MCU Digital Pin.  Again, see sketch comments.
 $Comp
 L power:GNDD #PWR?
@@
 Text Notes 10750 5000 1    60   Italic 12
 *See note
-Text Notes 9150 6450 0    56   ~ 11
-NOTE FOR MCU ANALOG PINS:  Low-\nnumbered Analog Input pins are reserved \nfor all existing DPOT-controlled leg outputs.  \nUnused Analog Pins above them may be\nused to display additional plotter traces\nwhen so defined in preprocessor macros.
+Text Notes 9150 6450 0    56   ~ 0
+*NOTE FOR MCU ANALOG PINS:  Low-\nnumbered Analog Input pins are reserved \nfor all existing DPOT-controlled leg outputs.  \nUnused Analog Pins above them may be\nused to display additional plotter traces\nwhen so defined in preprocessor macros.
 Text Notes 3650 3850 0    56   ~ 0
 NOTE: Decoupling C banks 1-2 each consist of a \n2-10 µF tantalum plus a low-ESR sub-µF capacitor \nwhich gets located in direct-as-practical path \nbetween + and GND pins of the active device \npaired with.

Commit message: Add files via upload
Other:
- note added: "NOTE: Additional matching MSB-level DPots are\nallowed in this P0W-P0B loop. Only a single \nLSB-level Dpot is allowed which must be of a\nresistance lower than or equal to MSB-level DPots.\nPins 5 and 6 are interchangeable, so the actual\nbuild will best wire them for the layout."
- note added: "NOTE: The LM334 devices must receive 5 VDC or greater due to their own operating voltage range. \nTheir functional range will be substantially limited if powered by the 3 or 3.3 VDC of many MCUs. \nProvide a dedicated positive power supply to them if 5 VDC is not otherwise available, then carefully \nensure the output levels from them are prevented from exceeding the input range of the remaining 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"
- note removed: "NOTE: Additional matching MSB-level DPots are\nallowed in this P0W-P0B loop. Only a single \nLSB-level Dpot is allowed which must be of a\nresistance lower than or equal to MSB-level DPots."
- note removed: "NOTE: The LM334 devices must receive 5 VDC or greater due to their own operating voltage range. \nTheir functional range will be substantially limited if powered by the 3 or 3.3 VDC of many MCUs. \nProvide a dedicated positive power supply to them if 5 VDC is not otherwise available, and carefully \nensure the output levels from them are prevented from exceeding the input range of the remaining \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"
Changed lines of the file:
@@
 Text GLabel 7550 4200 2    48   Input ~ 0
 <From_MCU_Digital_Pin_driving_this_CS
-Text Notes 3650 3050 0    59   ~ 0
-NOTE: Additional matching MSB-level DPots are\nallowed in this P0W-P0B loop.  Only a single \nLSB-level Dpot is allowed which must be of a\nresistance lower than or equal to MSB-level DPots.
+Text Notes 3650 3200 0    59   ~ 0
+NOTE: Additional matching MSB-level DPots are\nallowed in this P0W-P0B loop.  Only a single \nLSB-level Dpot is allowed which must be of a\nresistance lower than or equal to MSB-level DPots.\nPins 5 and 6 are interchangeable, so the actual\nbuild will best wire them for the layout.
 Text Notes 1000 3100 0    59   ~ 0
 NOTE: If convenient polarity flipping is desired,\n a 4-way house light switch  may be placed in \nthe electrode circuit between the electrodes and the \ncoaxial cable, assuming you hook it up correctly.
@@
 NOTE: Decoupling C banks 1-2 each consist of a \n2-10 µF tantalum plus a low-ESR sub-µF capacitor \nwhich gets located in direct-as-practical path \nbetween + and GND pins of the active device \npaired with.
 Text Notes 650  1300 0    66   ~ 0
-NOTE:  The LM334 devices must receive 5 VDC or greater due to their own operating voltage range.  \nTheir functional range will be substantially limited if powered by the 3 or 3.3 VDC of many MCUs.  \nProvide a dedicated positive power supply to them if 5 VDC is not otherwise available, and carefully \nensure the output levels from them are prevented from exceeding the input range of the remaining \ncircuitry.
+NOTE:  The LM334 devices must receive 5 VDC or greater due to their own operating voltage range.  \nTheir functional range will be substantially limited if powered by the 3 or 3.3 VDC of many MCUs.  \nProvide a dedicated positive power supply to them if 5 VDC is not otherwise available, then carefully \nensure the output levels from them are prevented from exceeding the input range of the remaining \ncircuitry.
 Text Notes 5450 7600 2    60   Italic 12
 *See note for the above DPot set
@@
 Wire Bus Line
 	6150 2600 6150 4400
-Wire Wire Line
-	1300 5350 1300 7100
-Wire Wire Line
-	4900 2500 6350 2500
-Wire Wire Line
-	4200 7050 6350 7050
-Wire Bus Line
-	8850 2000 8850 3300
-Wire Bus Line
-	4800 2600 6150 2600
-Wire Wire Line
-	1450 1950 2850 1950
-Wire Wire Line
-	1450 1550 2900 1550
-Wire Bus Line
-	4100 7150 6550 7150
-Wire Bus Line
-	7400 2000 7400 3300
-Wire Bus Line
-	10050 1700 10050 2500
 Text Notes 7300 7250 0    58   ~ 0
 1
+Wire Wire Line
+	1300 5350 1300 7100
+Wire Wire Line
+	4900 2500 6350 2500
+Wire Wire Line
+	4200 7050 6350 7050
+Wire Bus Line
+	8850 2000 8850 3300
+Wire Bus Line
+	4800 2600 6150 2600
+Wire Wire Line
+	1450 1950 2850 1950
+Wire Wire Line
+	1450 1550 2900 1550
+Wire Bus Line
+	4100 7150 6550 7150
+Wire Bus Line
+	7400 2000 7400 3300
+Wire Bus Line
+	10050 1700 10050 2500
 $EndSCHEMATC

Commit message: Add files via upload
Connections:
- wire segments 92 -> 90
Other:
- note added: "NOTE: Additional matching MSB-level DPots are\nallowed in this P0W-P0B loop. Only a single \nLSB-level Dpot is allowed which must be of a\nresistance lower than or equal to MSB-level DPots.\nPins 5 and 6 are interchangeable, so the actual\nconnect order will be layout-dependent."
- note added: "NOTE: Capacitor banks 1 & 2 each consist of a \n2-10 µF tantalum plus a low-ESR sub-µF capacitor \nwhich gets located in direct-as-practical path be-\ntween Vcc of one device to GND of the other device. \nNOT SHOWN: One decoupling capacitor bank of same \nvalues for all digital parts combined."
- note removed: "NOTE: Additional matching MSB-level DPots are\nallowed in this P0W-P0B loop. Only a single \nLSB-level Dpot is allowed which must be of a\nresistance lower than or equal to MSB-level DPots.\nPins 5 and 6 are interchangeable, so the actual\nbuild will best wire them for the layout."
- note removed: "NOTE: Decoupling C banks 1-2 each consist of a \n2-10 µF tantalum plus a low-ESR sub-µF capacitor \nwhich gets located in direct-as-practical path \nbetween + and GND pins of the active device \npaired with."
Changed lines of the file:
@@
 <From_MCU_Digital_Pin_driving_this_CS
 Text Notes 3650 3200 0    59   ~ 0
-NOTE: Additional matching MSB-level DPots are\nallowed in this P0W-P0B loop.  Only a single \nLSB-level Dpot is allowed which must be of a\nresistance lower than or equal to MSB-level DPots.\nPins 5 and 6 are interchangeable, so the actual\nbuild will best wire them for the layout.
+NOTE: Additional matching MSB-level DPots are\nallowed in this P0W-P0B loop.  Only a single \nLSB-level Dpot is allowed which must be of a\nresistance lower than or equal to MSB-level DPots.\nPins 5 and 6 are interchangeable, so the actual\nconnect order will be layout-dependent.
 Text Notes 1000 3100 0    59   ~ 0
 NOTE: If convenient polarity flipping is desired,\n a 4-way house light switch  may be placed in \nthe electrode circuit between the electrodes and the \ncoaxial cable, assuming you hook it up correctly.
@@
 L power:GNDA #PWR?
 U 1 1 5C193F33
-P 3000 4200
-F 0 "#PWR?" H 3000 3950 50  0001 C CNN
-F 1 "GNDA" H 3200 4150 50  0000 C CNN
-F 2 "" H 3000 4200 50  0001 C CNN
-F 3 "" H 3000 4200 50  0001 C CNN
-	1    3000 4200
+P 2250 3700
+F 0 "#PWR?" H 2250 3450 50  0001 C CNN
+F 1 "GNDA" H 2250 3550 50  0000 C CNN
+F 2 "" H 2250 3700 50  0001 C CNN
+F 3 "" H 2250 3700 50  0001 C CNN
+	1    2250 3700
 	1    0    0    -1
 $EndComp
@@
 L power:VCC #PWR?
 U 1 1 5C19D6AB
-P 5250 4300
-F 0 "#PWR?" H 5250 4150 50  0001 C CNN
-F 1 "VCC" H 5267 4473 50  0000 C CNN
-F 2 "" H 5250 4300 50  0001 C CNN
-F 3 "" H 5250 4300 50  0001 C CNN
-	1    5250 4300
+P 5250 4200
+F 0 "#PWR?" H 5250 4050 50  0001 C CNN
+F 1 "VCC" H 5267 4373 50  0000 C CNN
+F 2 "" H 5250 4200 50  0001 C CNN
+F 3 "" H 5250 4200 50  0001 C CNN
+	1    5250 4200
 	1    0    0    -1
 $EndComp
@@
 $EndComp
 $Comp
-L power:GNDD #PWR?
-U 1 1 5C1C4E62
-P 4700 4300
-F 0 "#PWR?" H 4700 4050 50  0001 C CNN
-F 1 "GNDD" H 4704 4145 50  0000 C CNN
-F 2 "" H 4700 4300 50  0001 C CNN
-F 3 "" H 4700 4300 50  0001 C CNN
-	1    4700 4300
-	1    0    0    -1
-$EndComp
-$Comp
 L Device:C_Small C2_bank
 U 1 1 5C1C5AE4
@@
 	0    1    1    0
 $EndComp
-$Comp
-L power:GNDD #PWR?
-U 1 1 5C1C6E06
-P 2250 3700
-F 0 "#PWR?" H 2250 3450 50  0001 C CNN
-F 1 "GNDD" H 2250 3550 50  0000 C CNN
-F 2 "" H 2250 3700 50  0001 C CNN
-F 3 "" H 2250 3700 50  0001 C CNN
-	1    2250 3700
-	1    0    0    -1
-$EndComp
 Wire Wire Line
 	10350 4450 10500 4450
@@
 Text Notes 9150 6450 0    56   ~ 0
 *NOTE FOR MCU ANALOG PINS:  Low-\nnumbered Analog Input pins are reserved \nfor all existing DPOT-controlled leg outputs.  \nUnused Analog Pins above them may be\nused to display additional plotter traces\nwhen so defined in preprocessor macros.
-Text Notes 3650 3850 0    56   ~ 0
-NOTE: Decoupling C banks 1-2 each consist of a \n2-10 µF tantalum plus a low-ESR sub-µF capacitor \nwhich gets located in direct-as-practical path \nbetween + and GND pins of the active device \npaired with.
+Text Notes 3650 3950 0    56   ~ 0
+NOTE: Capacitor banks 1 & 2 each consist of a \n2-10 µF tantalum plus a low-ESR sub-µF capacitor \nwhich gets located in direct-as-practical path be-\ntween Vcc of one device to GND of the other device.  \nNOT SHOWN: One decoupling capacitor bank of same \nvalues for all digital parts combined.
 Text Notes 650  1300 0    66   ~ 0
 NOTE:  The LM334 devices must receive 5 VDC or greater due to their own operating voltage range.  \nTheir functional range will be substantially limited if powered by the 3 or 3.3 VDC of many MCUs.  \nProvide a dedicated positive power supply to them if 5 VDC is not otherwise available, then carefully \nensure the output levels from them are prevented from exceeding the input range of the remaining \ncircuitry.
@@
 Wire Wire Line
 	4800 4300 4700 4300
-Wire Wire Line
-	5250 4300 5250 4350
-Connection ~ 5250 4300
-Wire Wire Line
-	5000 4300 5250 4300
 Connection ~ 2900 6900
 Entry Wire Line
@@
 	2900 6900 2900 7150
 Wire Wire Line
-	2450 3600 2500 3600
-Wire Wire Line
 	2900 1550 2900 2150
 Wire Wire Line
@@
 Wire Wire Line
 	6350 7050 6350 5200
-Connection ~ 2500 3600
-Wire Wire Line
-	2500 3600 2600 3600
 Connection ~ 4250 4600
 Wire Wire Line
 	4250 4600 4250 5600
-Wire Wire Line
-	2350 4000 2400 4000
 Wire Wire Line
 	2100 4000 2400 4000
@@
 1
 Wire Wire Line
+	2500 3600 2600 3600
+Wire Wire Line
+	5250 4200 5250 4300
+Wire Wire Line
+	5000 4300 5250 4300
+Connection ~ 5250 4300
+$Comp
+L power:GNDA #PWR?
+U 1 1 5C1E5690
+P 3000 4200
+F 0 "#PWR?" H 3000 3950 50  0001 C CNN
+F 1 "GNDA" H 3150 4100 50  0000 C CNN
+F 2 "" H 3000 4200 50  0001 C CNN
+F 3 "" H 3000 4200 50  0001 C CNN
+	1    3000 4200
+	1    0    0    -1
+$EndComp
+$Comp
+L power:GNDA #PWR?
+U 1 1 5C1E56EB
+P 4700 4300
+F 0 "#PWR?" H 4700 4050 50  0001 C CNN
+F 1 "GNDA" H 4705 4127 50  0000 C CNN
+F 2 "" H 4700 4300 50  0001 C CNN
+F 3 "" H 4700 4300 50  0001 C CNN
+	1    4700 4300
+	1    0    0    -1
+$EndComp
+Wire Wire Line
 	1300 5350 1300 7100
