File: embeddeds/GWAAM-Sea Training Aid.sch (KiCad schematic (older format))
At the start: 19 parts, among them J1 Conn_Coaxial, U1 LM334Z, U2 LM334Z, U3-A , U3-B U3_AD8244ARMZ, U3-C U3_AD8244ARMZ, U3-D U3_AD8244ARMZ, U4 74LV138 only needed with larg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, U5... 74LV138 only for large number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

Commit message: Add files via upload
Parts:
- removed U1: LM334Z, Package_TO_SOT_THT:TO-92_Inline, symbol Reference_Current:LM334Z
- added C1: 0.1 µF, symbol Device:C
- added J2: Conn_Coaxial, symbol Connector:Conn_Coaxial
- added R1: 22KΩ, symbol Device:R_US
- renumbered R1 to R2
Connections:
- net labels added: Off-board_coaxial_cables_x2
- net labels removed: Off-board_coaxial_cable
- wire segments 88 -> 92
Other:
- note added: "15 Jan 2019 (C) Copyright Kenneth L. Anderson 2019"
- note added: "GWAAMC Training Aid - System Diagram"
- note added: "NOTE: If convenient polarity flipping is desired,\n a 4-way house light switch may be placed \nin the electrode circuit between the electrodes and \nthe coaxial cable, assuming you hook it up correctly."
- note added: "NOTE: Sketch-adjustable to \nccommodate sweet-spot \nreference level specific to \nselected ADC"
- note added: "NOTE: The LM334 devices must receive 5 VDC or greater due to their own operating voltage range. Their \nfunctional range will be substantially limited if powered by the 3 or 3.3 VDC of many MCUs. Provide a \ndedicated positive power supply to them if 5 VDC is not otherwise available, then carefully ensure the output \nlevels from them are prevented from exceeding the input range of the remaining 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"
- note added: "To-be-determined: \nhigh impedance, \nadjustable, constant \ncurrent sink which can \nutilize the DPot1 bank \nleftover from previous \ndesign that used \nLM334. \n\n\n 1.5-2.5 Vdc high \n impedance range\n\n .15-2.5 µA adj."
- note removed: "18 Dec 2018"
- note removed: "GWAAMC Training Aid"
- note removed: "NOTE: If convenient polarity flipping is desired,\n a 4-way house light switch may be placed in \nthe electrode circuit between the electrodes and the \ncoaxial cable, assuming you hook it up correctly."
- note removed: "NOTE: The LM334 devices must receive 5 VDC or greater due to their own operating voltage range. \nTheir functional range will be substantially limited if powered by the 3 or 3.3 VDC of many MCUs. \nProvide a dedicated positive power supply to them if 5 VDC is not otherwise available, then carefully \nensure the output levels from them are prevented from exceeding the input range of the remaining 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"
- moved on the sheet: J1
