File: embeddeds/uno shield.kicad_pcb (KiCad board)
At the start: 2 copper layers, 68.6 x 53.3 mm, 58 parts, among them J1 Conn_3.5mm, J2 Power, J3 Analog, J4 Digital, J5 Digital, J6 Conn_01x04_Female, P1 CONN_01X01, P2 CONN_01X01, P3 CONN_01X01, P4 CONN_01X01, Q1 MMBF5462 (2N5462), Q2 MMBF5462 (2N5462), Q3 DMN601K-7, Q4 DMN601K-7, Q5 DMN601K-7, Q6 DMN601K-7, Q7 DMN601K-7, U1 AD8244ARMZ, U2 ADL5315ACPZ-R7, U3 REF200AU, U4 LM334M, U5 LM334M, U6 MCP4262-502E_UN, U7 MCP4262-104E_UN

Commit message: This file contains some or entire project in Kicad
Parts:
- removed J6: Conn_01x04_Female, multipackage:FFC_2x02_P2.00mm_Vertical
- added J6_A7,A6: Conn_01x02_gender_unknown, Connector_PinHeader_2.54mm:PinHeader_1x02_P2.54mm_Vertical, B.Cu at (175.4, 120.3)
- added J7_A7,A6: Conn_01x02_Female, Connector_PinHeader_2.54mm:PinHeader_1x02_P2.54mm_Vertical, B.Cu at (171.1, 119.1)
- moved J1 2.84 mm to (175.5, 113.6)
- moved R9 1.40 mm to (134.6, 112.5)
- moved Q1 0.96 mm to (140.1, 107.6)
- moved U7 0.86 mm to (163.6, 104.6)
- moved R8 0.75 mm to (162.2, 108.0)
- moved U6 0.71 mm to (163.6, 104.7)
- moved JP2 0.41 mm to (169.4, 109.5), turned to 0 degrees
Connections:
- Q2 pad 2: Net-(JP2-Pad1) -> Net-(JP2-Pad2)
- R8 pad 2: Net-(JP2-Pad2) -> Net-(JP2-Pad1)
- U5 pad 2: Net-(JP2-Pad1) -> Net-(JP2-Pad2)
- U5 pad 3: Net-(JP2-Pad1) -> Net-(JP2-Pad2)
- U6 pad 5: Net-(JP2-Pad1) -> Net-(JP2-Pad2)
Routing:
- net /A6: track 32.1 -> 91.1 mm, vias 0 -> 3
- net Net-(JP2-Pad2): track 3.41 -> 49.2 mm, vias 0 -> 4
- net Net-(JP2-Pad1): track 52.0 -> 9.18 mm, vias 4 -> 0
- net /1st_stage_guard_trace: track 374.5 -> 406.9 mm, vias 12 -> 16
- net /A7: track 63.5 -> 93.9 mm, vias 6 -> 8
- net GNDD: track 270.6 -> 250.6 mm, vias 7 -> 9
- net GNDA: track 115.1 -> 129.8 mm, vias 18 -> 19
- net /A0: track 105.3 -> 108.6 mm
- net /3(**): track 14.8 -> 17.9 mm, vias 0 -> 1
- net /2: track 17.5 -> 20.5 mm, vias 0 -> 1
- net /3rd_stage_guard_trace: track 15.4 -> 18.0 mm
- net /5(**): track 38.7 -> 36.4 mm
- net Net-(C1-Pad1): track 24.1 -> 26.3 mm
- net Net-(C2-Pad2): track 6.18 -> 4.05 mm
- net Net-(U5-Pad1): track 25.2 -> 23.8 mm
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- added copper zone on B.Cu, net GNDD
- removed copper zone on B.Cu, net (none)
Other:
- board text added: "!"
- board text added: "!!!YOU MUST CONFIGURE JP1,JP3: (on this side is reversible) SOLDER PADS 1 TO 2 ON BOTH UNLESS INFORMED THAT EXPERIMENTAL PADS 2 TO 3 WORK BETTER! ON THIS SIDE FOR EASY REVERSAL"
- board text added: "2 JP3 3 1"
- board text added: "3 JP1 1 2"
- board text added: "CONSTANTLY CHECK BOARD CLEARANCES MATING W/MCU"
- board text added: "ENSURE AIRTIGHTNESS UNDER THE SHIELD: Solder seal the shield's vias from this side & include affixed under the shield the dried dessicant pkg you received with U3. Solder ENTIRE shield rim after soldering JP1 and JP3 and placing compo- nents. Purpose: U3 is a high precision device that can be detrimentally affected by its plastic package absorbing the same moisture that all plastic components abs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"
- board text added: "Expect mistakes each step. Check that often to protect your sanity later"
- board text added: "J7"
- board text added: "JP2"
- board text added: "JP3"
- board text added: "Other side"
- board text removed: "!!!INSIDE THE SHIELD YOU MUST CONFIGURE JP1,JP3: SOLDER PADS 1 TO 2 ON BOTH UNLESS INFORMED THAT EXPERIMENTAL PADS 2 TO 3 WORK BETTER!!!!"
- board text removed: "ALWAYS ENSURE BOARD CLEARANCES MATING W/MCU"
- board text removed: "ENSURE AIRTIGHTNESS UNDER THE SHIELD: Solder seal the shield's vias from this side & include affixed under the shield the dried dessicant pkg you received with U1. Solder ENTIRE shield rim after soldering JP1 and JP3 and placing compo- nents. Purpose: U1 is a high precision device that can be detrimentally affected by its plastic package absorbing the same moisture that all plastic components abs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"
- board text removed: "Expect mistakes each step. Check that often to protect your sanity"
- board text removed: "Trim protruding < ends as needed before soldering"
