File: uno shield.kicad_pcb (KiCad board)
At the start: 2 copper layers, 68.6 x 53.3 mm, 58 parts, among them J1 Conn_3.5mm, J2 Power, J3 Analog, J4 Digital, J5 Digital, J6_A6,A7 Conn_01x02_Female, P1 CONN_01X01, P2 CONN_01X01, P3 CONN_01X01, P4 CONN_01X01, Q1 MMBF5462 (2N5462), Q2 MMBF5462 (2N5462), Q3 DMN601K-7, Q4 DMN601K-7, Q5 DMN601K-7, Q6 DMN601K-7, Q7 DMN601K-7, U1 AD8244ARMZ, U2 ADL5315ACPZ-R7, U3 REF200AU, U4 LM334M, U5 LM334M, U6 MCP4262-502E_UN, U7 MCP4262-104E_UN

Commit message: Kicad project files
Parts:
- added J7_A7,A6: Conn_01x02_Female, Connector_PinHeader_2.54mm:PinHeader_1x02_P2.54mm_Vertical, B.Cu at (171.1, 119.1)
- J6_A7,A6: renamed from J6_A6,A7; value Conn_01x02_Female -> Conn_01x02_gender_unknown
- moved J1 2.24 mm to (175.5, 113.6)
- moved U7 0.86 mm to (163.6, 104.6)
- moved J6_A7,A6 0.80 mm to (175.4, 120.3)
- moved R8 0.75 mm to (162.2, 108.0)
- moved U6 0.71 mm to (163.6, 104.7)
- moved JP2 0.41 mm to (169.4, 109.5)
Connections:
- Q2 pad 2: Net-(JP2-Pad1) -> Net-(JP2-Pad2)
- R8 pad 2: Net-(JP2-Pad2) -> Net-(JP2-Pad1)
- U5 pad 2: Net-(JP2-Pad1) -> Net-(JP2-Pad2)
- U5 pad 3: Net-(JP2-Pad1) -> Net-(JP2-Pad2)
- U6 pad 5: Net-(JP2-Pad1) -> Net-(JP2-Pad2)
Routing:
- net Net-(JP2-Pad2): track 6.49 -> 49.2 mm, vias 1 -> 4
- net Net-(JP2-Pad1): track 50.9 -> 9.18 mm, vias 4 -> 0
- net GNDD: track 270.7 -> 250.6 mm, vias 7 -> 9
- net /1st_stage_guard_trace: track 390.0 -> 406.9 mm, vias 12 -> 16
- net +5V: track 297.9 -> 284.9 mm
- net /A6: track 85.5 -> 91.1 mm
- net /3(**): track 14.8 -> 17.9 mm, vias 0 -> 1
- net /2: track 17.5 -> 20.5 mm, vias 0 -> 1
- net /5(**): track 39.0 -> 36.4 mm
- net GNDA: track 132.0 -> 129.8 mm, vias 18 -> 19
- net Net-(C2-Pad2): track 6.18 -> 4.05 mm
- net Net-(J1-PadS): track 29.1 -> 31.1 mm
- net Net-(C1-Pad1): track 24.5 -> 26.3 mm
- net /A7: track 92.3 -> 93.9 mm, vias 7 -> 8
- net Net-(U5-Pad1): track 25.2 -> 23.8 mm
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Other:
- board text added: "!"
- board text added: "!!!YOU MUST CONFIGURE JP1,JP3: (on this side is reversible) SOLDER PADS 1 TO 2 ON BOTH UNLESS INFORMED THAT EXPERIMENTAL PADS 2 TO 3 WORK BETTER! ON THIS SIDE FOR EASY REVERSAL"
- board text added: "2 JP3 3 1"
- board text added: "3 JP1 1 2"
- board text added: "CONSTANTLY CHECK BOARD CLEARANCES MATING W/MCU"
- board text added: "ENSURE AIRTIGHTNESS UNDER THE SHIELD: Solder seal the shield's vias from this side & include affixed under the shield the dried dessicant pkg you received with U3. Solder ENTIRE shield rim after soldering JP1 and JP3 and placing compo- nents. Purpose: U3 is a high precision device that can be detrimentally affected by its plastic package absorbing the same moisture that all plastic components abs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"
- board text added: "J7"
- board text added: "JP3"
- board text added: "Other side"
- board text removed: "!!!INSIDE THE SHIELD YOU MUST CONFIGURE JP1,JP3: SOLDER PADS 1 TO 2 ON BOTH UNLESS INFORMED THAT EXPERIMENTAL PADS 2 TO 3 WORK BETTER!!!!"
- board text removed: "A7 A6 proximity on many MCUs"
- board text removed: "ALWAYS ENSURE BOARD CLEARANCES MATING W/MCU"
- board text removed: "ENSURE AIRTIGHTNESS UNDER THE SHIELD: Solder seal the shield's vias from this side & include affixed under the shield the dried dessicant pkg you received with U1. Solder ENTIRE shield rim after soldering JP1 and JP3 and placing compo- nents. Purpose: U1 is a high precision device that can be detrimentally affected by its plastic package absorbing the same moisture that all plastic components abs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"
- board text removed: "Trim protruding < ends as needed before soldering"

Commit message: Add files via upload
Parts:
- removed J7_A7,A6: Conn_01x02_Female, Connector_PinHeader_2.54mm:PinHeader_1x02_P2.54mm_Vertical
- added J7_A7,A1: Conn_01x02_Female, Connector_PinHeader_2.54mm:PinHeader_1x02_P2.54mm_Vertical, B.Cu at (170.4, 119.3)
- JP1: moved to B.Cu
- JP2: renamed from JP3; moved to B.Cu
- Q3, Q4, Q5, Q6, Q7: moved to F.Cu
- U2: value ADL5315ACPZ-R7 -> ADL5315
- moved Q4 12.9 mm to (132.2, 88.5), turned to 180 degrees
- moved Q6 11.0 mm to (122.5, 89.8), turned to 180 degrees
- moved Q5 10.9 mm to (122.5, 93.3), turned to 0 degrees
- moved Q7 10.8 mm to (122.5, 86.3), turned to 180 degrees
- moved Q3 10.7 mm to (132.2, 92.0)
- moved JP2 0.38 mm to (142.6, 122.7)
- moved J1 0.31 mm to (175.2, 113.7)
- moved R12 0.26 mm to (120.3, 84.3)
- renumbered J6_A7,A6 to J6_A7,A1, JP2 to JP3
Connections:
- U2 pad 7: (no net) -> /2nd_stage_guard_trace
- U2 pad 9: (no net) -> GNDA
Routing:
- net GNDD: track 250.6 -> 214.1 mm, vias 9 -> 20
- net +5V: track 284.9 -> 255.2 mm, vias 22 -> 20
- net GNDA: track 129.8 -> 156.5 mm, vias 19 -> 21
- net Net-(Q3-Pad3): track 5.60 -> 23.8 mm, vias 2 -> 4
- net Net-(Q3-Pad2): track 73.3 -> 89.2 mm, vias 4 -> 5
- net /7: track 55.9 -> 42.1 mm, vias 1 -> 2
- net Net-(D3-Pad1): track 3.24 -> 13.8 mm, vias 0 -> 1
- net /6(**): track 54.5 -> 45.0 mm, vias 7 -> 8
- net Net-(D1-Pad1): track 14.3 -> 22.8 mm, vias 0 -> 3
- net /1st_stage_guard_trace: track 406.9 -> 398.5 mm
- net Net-(D2-Pad1): track 4.18 -> 8.16 mm, vias 0 -> 2
- net Net-(U5-Pad1): track 23.8 -> 21.1 mm
- net /A0: track 108.6 -> 107.4 mm
- net /A6: track 91.1 -> 92.3 mm
- net Net-(C2-Pad2): track 4.05 -> 5.05 mm
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Other:
- board text added: "!! JP1,2: Solder across pads 1 and 2 unless informed that 2 to 3 works!"
- board text added: "!!!YOU MUST CONFIGURE JP1,JP2: (on this side is reversible) SOLDER PADS 1 TO 2 ON BOTH UNLESS INFORMED THAT EXPERIMENTAL PADS 2 TO 3 WORK BETTER! ON THIS SIDE FOR EASY REVERSAL"
- board text added: "Arduino UNO Extension Board Rev. 06 SMD (C) June 2019 A Reviving Civility Matt. 21:21"
- board text added: "ENSURE AIRTIGHTNESS UNDER THE SHIELD: Solder seal the shield's vias from this side & include affixed under the shield the dried dessi- cant pkg you received with U2. Solder ENTIRE shield rim after soldering JP1 and JP2 and plac- ing com- ponents. Purpose: U2 is a high precision device that can be affected detrimentally by its plastic pack- age absorbing the same moisture that all plastic componen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"
- board text removed: "!! JP1,3: Solder across pads 1 and 2 unless informed that 2 to 3 works!"
- board text removed: "!!!YOU MUST CONFIGURE JP1,JP3: (on this side is reversible) SOLDER PADS 1 TO 2 ON BOTH UNLESS INFORMED THAT EXPERIMENTAL PADS 2 TO 3 WORK BETTER! ON THIS SIDE FOR EASY REVERSAL"
- board text removed: "2 JP3 3 1"
- board text removed: "3 JP1 1 2"
- board text removed: "Arduino UNO Extension Board Rev. 06 (C) June 2019 A Reviving Civility Matt. 21:21"
- board text removed: "C3"
- board text removed: "ENSURE AIRTIGHTNESS UNDER THE SHIELD: Solder seal the shield's vias from this side & include affixed under the shield the dried dessicant pkg you received with U3. Solder ENTIRE shield rim after soldering JP1 and JP3 and placing compo- nents. Purpose: U3 is a high precision device that can be detrimentally affected by its plastic package absorbing the same moisture that all plastic components abs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"
- board text removed: "Other side"
