File: uno shield.sch (KiCad schematic (older format))
At the start: 58 parts, among them J1 Conn_3.5mm, J2 Power, J3 Analog, J4 Digital, J5 Digital, J6_A6,A7 Conn_01x02_Female, P1 CONN_01X01, P2 CONN_01X01, P3 CONN_01X01, P4 CONN_01X01, Q1 MMBF5462 (2N5462), Q2 MMBF5462 (2N5462), Q3 DMN601K-7, Q4 DMN601K-7, Q5 DMN601K-7, Q6 DMN601K-7, Q7 DMN601K-7, U1 AD8244ARMZ, U2 ADL5315ACPZ-R7, U3 REF200AU, U4 LM334M, U5 LM334M, U6 MCP4262-502E_UN, U7 MCP4262-104E_UN

Commit message: Add files via upload
Parts:
- added J7_A7,A1: Conn_01x02_Female, Connector_PinHeader_2.54mm:PinHeader_1x02_P2.54mm_Vertical, symbol Connector:Conn_01x02_Female
- J6_A7,A1: renamed from J6_A6,A7; value Conn_01x02_Female -> Conn_01x02_gender_unknown; Part_number (none) -> male: part of a second TSW-150-05-T-S/4-103327-0 female: SS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
- JP1: ClickToSortForPlacement (none) -> 00 Pads 2-3 were experimental. Solder-short pads 1 to 2 unl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
- JP2: renamed from JP3; ClickToSortForPlacement (none) -> 00 Pads 2-3 were experimental. Solder-short pads 1 to 2 unl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
- Q1, Q2: ClickToSortForPlacement 00 Not component, only use temporary solder bridge on board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 -> (none)
- SHLD1: Part_number MS263-20 (just the cover) -> MS263-20 (will only use the cover to keep hermetic sealed)
- U1: ClickToSortForPlacement 00 00 !Assembly instructions not complete - do not trust th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 -> 02 Place (always means solder herein), then check work for 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
- U2: ClickToSortForPlacement (none) -> 00 00 !Assembly instructions are not yet complete - do not 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
- U3: Part_number REF200AU -> REF200AU (will contain dessicant you'll need to place under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
- VR3, VR4: Part_number User/developer (\"hacker\") use only: PTV09A-4030U-B204 or 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 -> User/developer use only: PTV09A-4030U-B204 or may end in B2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
- renumbered JP2 to JP3
Connections:
- net 2nd_stage_guard_trace: now also U2.7 (SHLD)
- net A6: now also J7_A7,A1.2 (Pin_2)
- net A7: now also J7_A7,A1.1 (Pin_1)
- net GNDA: now also U2.9 (COMM)
- net at Q2.2 (D), U5.2, U5.3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: now also JP3.2 (B); no longer JP3.1 (A)
- net at R8.2: now also JP3.1 (A); no longer JP3.2 (B)
Other:
- note added: "GNDA used for \nguard trace between\nS and R1"
- note added: "When used as designed (body \nsoldered to PCB and cover used \nremoveably) the height of this \nshield is 10mm and not hermetically \nsealed.\n\nInstead, hermetic sealing is \nsuggested to provide you with \nthe ultimate in long term \nsensitivity stability in scientific\ninstrumentation class useages,\nwhich will also benefit from J1\nbeing a triax connector instead\nof the phone connector shown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"
- note added: "With triax cabling employed \n (not shown) guard trace will \n join to cable's guard \n conductor"
- note removed: "GNDA used for guard trace here"
- note removed: "When used as designed (body \nsoldered to PCB and cover used \nremoveably) the height of this \nshield is 10mm and not hermetically \nsealed.\n\nInstead, hermetic sealing is \nsuggested to provide you with \nthe ultimate in long term \nsensitivity stability.\n\nHermetic sealing is achieved by: \n\n#1) Solder sealing all micro-vias of\nthe PCB under the shield, and\n\n#2) not using the shield body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"
- moved on the sheet: R1, R4, SHLD1
