File: Where to find everything for making your own GWAAMC device/Files you need relative to the printed circuit board/Rev 8 in progress/Coax Cable and Diagnostic DUT.sch (KiCad schematic (older format))
At the start: 13 parts, among them J7 AudioJack2, J8 Cable end 2mm female, P10 Diagnostic DUT, P11 Conn_01x01_Male, P12 3.5mm_TRS_male_cable_end, P13 3.5mm_TRS_male_cable_end, P5 Conn_01x01_Male, P6 Dummy DUT, P7 Cable end 2mm male, P8 Cable end 2mm male, P9 Conn_01x01_Male

Commit message: Untested while awaiting bare PCB boards....
These KiCad and zipped gerber files are fully designed but not yet tested while I await the bare boards on order now.  I'm estimating mid- to late-October will see the final evaluation of operation of the entire device.  Shortly after that, I would expect to demonstrate its concepts and operation via YouTube and personal travel.
Parts:
- J8, P7, P8: Source http://www.digikey.com -> http://digikey.com
Changed lines of the file:
@@
 F 2 "Connector_PinHeader_1.00mm:PinHeader_1x01_P1.00mm_Horizontal" H 5300 4400 50  0001 C CNN
 F 3 "~" H 5300 4400 50  0001 C CNN
-F 4 "http://www.digikey.com" H 5300 4400 50  0001 C CNN "Source"
+F 4 "http://digikey.com" H 5300 4400 50  0001 C CNN "Source"
 F 5 "99" H 5300 4400 50  0001 C CNN "ClickToSortForPlacement"
 F 6 " CT3098-2-ND" H 5300 4400 50  0001 C CNN "Part_number"
@@
 F 4 "99" H 5025 4300 50  0001 C CNN "ClickToSortForPlacement"
 F 5 "CT3095-2-ND" H 5025 4300 50  0001 C CNN "Part_number"
-F 6 "http://www.digikey.com" H 5025 4300 50  0001 C CNN "Source"
+F 6 "http://digikey.com" H 5025 4300 50  0001 C CNN "Source"
 	1    5025 4300
 	0    1    1    0
@@
 F 2 "Connector_PinHeader_1.00mm:PinHeader_1x01_P1.00mm_Horizontal" H 4800 4400 50  0001 C CNN
 F 3 "~" H 4800 4400 50  0001 C CNN
-F 4 "http://www.digikey.com" H 4800 4400 50  0001 C CNN "Source"
+F 4 "http://digikey.com" H 4800 4400 50  0001 C CNN "Source"
 F 5 " CT3098-2-ND" H 4800 4400 50  0001 C CNN "Part_number"
 F 6 "99" H 4800 4400 50  0001 C CNN "ClickToSortForPlacement"
